File: schematics/01-valve-control/relay-bank/relay-bank.kicad_sch (KiCad schematic)
At the start: 6 parts, among them J102 PWR, J103 EN

Commit message: Add connector for valve control enable inputs
Parts:
- J103: footprint (none) -> royale:Molex_Nano-Fit_105313-xx05_1x05_P2.50mm_Horizontal
Changed lines of the file:
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@@
     (property "Reference" "J103" (id 0) (at 98.425 110.49 0))
     (property "Value" "EN" (id 1) (at 98.425 113.03 0))
-    (property "Footprint" "" (id 2) (at 98.425 121.92 0)
+    (property "Footprint" "royale:Molex_Nano-Fit_105313-xx05_1x05_P2.50mm_Horizontal" (id 2) (at 98.425 121.92 0)
       (effects (font (size 1.27 1.27)) hide)
     )
@@
     )
     (path "/6a7410ac-6f2d-41b6-9ae5-119b71f0d7e5"
-      (reference "J103") (unit 1) (value "EN") (footprint "")
+      (reference "J103") (unit 1) (value "EN") (footprint "royale:Molex_Nano-Fit_105313-xx05_1x05_P2.50mm_Horizontal")
     )
     (path "/00000000-0000-0000-0000-000061acc4fd/f741d2a6-3cfd-425c-b5b1-c8b6c7563112"

Commit message: Relay bank changes for manufacture
Parts:
- J102: Farnell (none) -> 2820686
- J103: Farnell (none) -> 3862799
Changed lines of the file:
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@@
+      (effects (font (size 1.27 1.27)) hide)
+    )
+    (property "Farnell" "~" (id 4) (at 100.33 88.9 0)
       (effects (font (size 1.27 1.27)) hide)
     )
@@
     )
     (property "Datasheet" "~" (id 3) (at 95.885 60.96 0)
+      (effects (font (size 1.27 1.27)) hide)
+    )
+    (property "Farnell" "2820686" (id 4) (at 95.885 60.96 0)
       (effects (font (size 1.27 1.27)) hide)
     )
@@
     )
     (property "Datasheet" "~" (id 3) (at 98.425 121.92 0)
+      (effects (font (size 1.27 1.27)) hide)
+    )
+    (property "Farnell" "3862799" (id 4) (at 98.425 121.92 0)
       (effects (font (size 1.27 1.27)) hide)
     )
@@
       (effects (font (size 1.27 1.27)) hide)
     )
+    (property "Farnell" "~" (id 4) (at 115.57 88.9 0)
+      (effects (font (size 1.27 1.27)) hide)
+    )
     (pin "1")
   )
@@
     )
     (property "Datasheet" "~" (id 3) (at 107.95 88.9 0)
+      (effects (font (size 1.27 1.27)) hide)
+    )
+    (property "Farnell" "~" (id 4) (at 107.95 88.9 0)
       (effects (font (size 1.27 1.27)) hide)
     )
@@
       (effects (font (size 1.27 1.27)) hide)
     )
+    (property "Farnell" "~" (id 4) (at 92.71 88.9 0)
+      (effects (font (size 1.27 1.27)) hide)
+    )
