File: schematics/12-repeater/repeater.kicad_pcb (KiCad board)
At the start: 4 copper layers, 50 x 25 mm, 13 parts, among them J1 Cat5, J2 Mini-DIN, U1 PCA9600D

Commit message: Add silkscreen
Parts:
- added G***: LOGO, royale:cusf_worm, B.Cu at (135.6, 123.5)
Other:
- board text added: "C. Yiu M. Li A. Farquharson"
- board text added: "Designed by"
- board text added: "H. Franks B. Kwok T. Yam"
- board text added: "I2C Repeater, the {dblquote}Magic Box{dblquote}"
- board text added: "Mar 2022"

Commit message: Silkscreen tweaks for manufacture
Other:
- board text added: "March 2022"
- board text removed: "Mar 2022"
Changed lines of the file:
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@@
   (gr_line (start 119.1 128) (end 169.1 128) (layer "Edge.Cuts") (width 0.1))
   (gr_line (start 169.1 128) (end 169.1 103) (layer "Edge.Cuts") (width 0.1))
-  (gr_text "Designed by" (at 142.2 114.4) (layer "B.SilkS")
+  (gr_text "Designed by" (at 142.2 114.35) (layer "B.SilkS")
     (effects (font (size 0.5 0.5) (thickness 0.1)) (justify mirror))
   )
-  (gr_text "H. Franks\nB. Kwok\nT. Yam" (at 145.8 116.2) (layer "B.SilkS")
+  (gr_text "H. Franks\nB. Kwok\nT. Yam" (at 146.25 116.2) (layer "B.SilkS")
     (effects (font (size 0.5 0.5) (thickness 0.1)) (justify left mirror))
   )
-  (gr_text "C. Yiu\nM. Li\nA. Farquharson" (at 141.6 116.2) (layer "B.SilkS")
+  (gr_text "C. Yiu\nM. Li\nA. Farquharson" (at 141.85 116.2) (layer "B.SilkS")
     (effects (font (size 0.5 0.5) (thickness 0.1)) (justify left mirror))
   )
-  (gr_text "Mar 2022" (at 142.2 118.2) (layer "B.SilkS")
+  (gr_text "March 2022" (at 142.2 118.2) (layer "B.SilkS")
     (effects (font (size 0.5 0.5) (thickness 0.1)) (justify mirror))
   )
